File: m5stack_interface_board_feetech_sts.kicad_pcb (KiCad board)
At the start: 2 copper layers, 50 x 20 mm, 18 parts, among them J1 B2B-XH-A(LF)(SN), J2 B4B-PH-K-S(LF)(SN), J3 22035035, J4 22035035, Q1 2SA1162GR, U1 MAX3485, U2 AP7333-33SAG

Commit message: add PCBWay's logo and URL
Parts:
- added G***: LOGO, LOGO, B.Cu at (166.4, 125.9)
Other:
- board text added: "https://www.pcbway.com/"
